File: Electronic Design/KiCAD/KiCad Projects/STM32 PCB Design/STM32 PCB Design.kicad_pcb (KiCad board)
At the start: 2 copper layers, 52.3 x 32.3 mm, 35 parts

Commit message: Files
Parts:
- added G***: LOGO, LOGO, F.Cu at (77.8, 54.4)
Other:
- board text removed: "VOLT"
