File: Electronic Design/KiCAD/KiCad Projects/STM32 PCB Design/STM32 PCB Design.kicad_sch (KiCad schematic)
At the start: 35 parts, among them J1 USB_B_Micro, J2 Conn_01x04, J3 Conn_01x04, J4 Conn_01x04, J5 Conn_01x04, J6 Conn_01x04, J7 Conn_01x02, SW2 SW_Wuerth_450301014042, U1 STM32F103C8T6, U2 AMS1117-3.3, Y1 Crystal_GND24

Commit message: Files
Other:
- note added: "STM32 Hobby Breakout Board"
- note removed: "STM32 Hobby Breakout Board (Volt)"
