File: Electronic Design/KiCAD/KiCad Projects/USB3.0 To Gigabit Ethernet Adapter Design/USB3.0 To Gigabit Ethernet Adapter Design.kicad_sch (KiCad schematic)
At the start: 0 parts

Commit message: Project files
Parts:
- added C1, C15, C3: 22u, Capacitor_SMD:C_0402_1005Metric, symbol Device:C
- added C10, C2, C8, C9: 12p, Capacitor_SMD:C_0402_1005Metric, symbol Device:C
- added C11, C12, C13, C14, C16, C17, C18, C19, C20, C21, C22, C23, C24, C25, C26, C27, C4, C5: 1u, Capacitor_SMD:C_0402_1005Metric, symbol Device:C
- added C6, C7: 100n, Capacitor_SMD:C_0402_1005Metric, symbol Device:C
- added J1: 692221030100, 692221030100:692221030100, symbol 692221030100:692221030100
- added J2: HR911130A, HR911130A:HANRUN_HR911130A, symbol HR911130A:HR911130A
- added L1, L2: 4u7, Capacitor_SMD:C_0402_1005Metric, symbol Device:L
- added R1: 53k6, Resistor_SMD:R_0402_1005Metric, symbol Device:R
- added R10, R11, R12, R13, R9: 1k, Resistor_SMD:R_0402_1005Metric, symbol Device:R
- added R2, R4, R5, R6, R7: 12k, Resistor_SMD:R_0402_1005Metric, symbol Device:R
- added R3, R8: 0R, Resistor_SMD:R_0402_1005Metric, symbol Device:R
- added U1: LAN7800, Package_DFN_QFN:QFN-48-1EP_7x7mm_P0.5mm_EP5.7x5.7mm_ThermalVias, symbol LAN7800Y9X:LAN7800
- added U2: SwitchingIC, Package_TO_SOT_SMD:SOT-23-5, symbol SwitchingIC:SwitchingIC
- added U3: ESD700, ESD7008MUTAG:DIO_MG2040MUTAG, symbol ESD7008MUTAG:ESD7008MUTAG
- added Y1: Crystal_GND24, Crystal:Crystal_SMD_SeikoEpson_FA238-4Pin_3.2x2.5mm, symbol Device:Crystal_GND24
Connections:
- new net: C7.1, J1.6 (STDB_SSTX+), U3.5
- new net: C7.2, U1.29 (USB3_TXDM)
- new net: J1.2 (D-), U1.27 (USB2_DM), U3.2
- new net: J1.3 (D+), U1.26 (USB2_DP), U3.1
- new net: C6.1, J1.5 (STDB_SSTX-), U3.4
- new net: J1.8 (STDB_SSRX-), U1.31 (USB3_RXDP), U3.7
- new net: J1.9 (STDB_SSRX+), U1.32 (USB3_RXDM), U3.8
- new net: J1.S2, J1.SH
- new net: R4.2, U1.35 (RESET_N/PME_CLEAR)
- new net: J2.14 (SIG), R13.2
- new net: C2.2, R1.2, R2.1, U2.5 (FB)
- new net: C8.2, U1.40 (XI), Y1.1
- new net: C9.2, U1.41 (XO), Y1.3
- new net: C10.2, U1.48 (REF_FILT)
- new net: C6.2, U1.28 (USB3_TXDP)
- new net: L1.1, U2.3 (SW)
- new net: R5.2, U1.23 (VBUS_DET)
- new net: R6.2, U1.34 (TEST)
- new net: R7.2, U1.37 (USBRBIAS)
- new net: R9.2, U1.47 (REF_REXT)
- new net: J2.1 (VCC), R12.1
- new net: J2.11 (SIG), R11.2
- new net: R10.1, R9.1
- new net +1.2V: C22.1, C23.1, C24.1, L2.2, R8.1, U1.15 (VDD12_SW_FB), U1.21 (VDD12CORE), U1.42 (VDD12CORE)
- new net +1.2VA: C25.1, C26.1, C27.1, R8.2, U1.25 (VDD12A), U1.30 (VDD12A), U1.44 (VDD12A)
- new net +2V5: C17.1, C18.1, C19.1, C20.1, C21.1, U1.12 (VDD25A), U1.3 (VDD25A), U1.45 (VDD25_REG_OUT), U1.6 (VDD25A), U1.9 (VDD25A)
- new net +3.3V: C11.1, C12.1, C13.1, C14.1, C15.1, C16.1, C2.1, C3.1, L1.2, R1.1, R11.1, R12.2, R13.1, R4.1, R5.1, U1.14 (VDD_SW_IN), U1.20 (VDDVARIO), U1.36 (VDDVARIO), U1.38 (VDD33A), U1.39 (VDDVARIO), U1.46 (VDD33_REG_IN)
- new net +VBUS: C4.1, J1.1 (VBUS), R3.1, U3.10, U3.11
- new net +VBUSF: C1.1, C5.1, R3.2, U2.1 (EN), U2.4 (VIN)
- new net 13: L2.1, U1.13 (VDD12_SW_OUT)
- new net GND: C1.2, C10.1, C11.2, C12.2, C13.2, C14.2, C15.2, C16.2, C17.2, C18.2, C19.2, C20.2, C21.2, C22.2, C23.2, C24.2, C25.2, C26.2, C27.2, C3.2, C4.2, C5.2, C8.1, C9.1, J1.4 (GND), J1.7 (GND_DRAIN), J2.10 (GND), J2.S2 (SHIELD), J2.SH (SHIELD), R10.2, R2.2, R6.1, R7.1, U2.2 (GND), U3.13 (GND), U3.15 (GND), U3.17 (GND), U3.3 (GND), U3.6 (GND), U3.9 (GND), Y1.2 (G), Y1.4 (G)
- new net LED2: J2.12 (LED2), U1.24 (SUSPEND_N/LED2/GPIO5)
- new net LED3: J2.13 (LED3), U1.33 (LED3/GPIO6)
- new net MD0+: J2.2 (MD0+), U1.1 (TR0P)
- new net MD0-: J2.3 (MD0-), U1.2 (TR0N)
- new net MD1+: J2.4 (MD1+), U1.4 (TR1P)
- new net MD1-: J2.7 (MD1-), U1.5 (TR1N)
- new net MD2+: J2.5 (MD2+), U1.7 (TR2P)
- new net MD2-: J2.6 (MD2-), U1.8 (TR2N)
- new net MD3+: J2.8 (MD3+), U1.10 (TR3P)
- new net MD3-: J2.9 (MD3-), U1.11 (TR3N)
- no-connect marks 0 -> 7
Other:
- note added: "Decoupling & Power Distribution Network"
- note added: "Ethernet Port"
- note added: "LAN Controller"
- note added: "Main Power"
